Commit message: new file:   ballbot_base_link.urdf 	new file:   ballbot_floor.urdf 	modified:   resources/robots/ballbot/urdf/ballbot.urdf 	modified:   resources/robots/h1/urdf/h1.urdf 	new file:   resources/robots/pybullet_test.py 	modified:   scripts/data_process/grad_fit_ballbot.py 	modified:   scripts/data_process/grad_fit_ballbot_shape.py 	modified:   scripts/data_process/grad_fit_h1.py 	modified:   scripts/data_process/grad_fit_h1_shape.py 	new file:   scripts/joint_mokey_ballbot.py 	modified:   scripts/joint_monkey_h1.py 	modified:   scripts/mjcf_to_urdf.py 	modified:   scripts/vis/vis_motion.py 	modified:   test.ipynb

File: resources/robots/ballbot/urdf/ballbot.urdf (robot description, URDF)
Before this commit: robot ballbot_new_hgy, 48 links, 46 joints
Links:
- removed link ball
- removed link base
- removed link head
- removed link left_elbow
- removed link left_hand
- removed link left_shoulder_pitch
- removed link left_shoulder_roll
- removed link left_shoulder_yaw
- removed link neck
- removed link right_elbow
- removed link right_hand
- removed link right_shoulder_pitch
- removed link right_shoulder_roll
- removed link right_shoulder_yaw
- removed link torso
- added link ball_link, mass 3.021143163744471; collision mesh filename=../meshes/ball.stl scale=0.001 0.001 0.001; visual mesh filename=../meshes/ball.stl scale=0.001 0.001 0.001
- added link ball_x_link, mass 0.01
- added link ball_y_link, mass 0.01
- added link base_link, mass 4.8833491952093615; collision mesh filename=../meshes/base.stl scale=0.001 0.001 0.001; visual mesh filename=../meshes/base.stl scale=0.001 0.001 0.001
- added link head_link, mass 1.0299685988699756; collision mesh filename=../meshes/head.stl scale=0.001 0.001 0.001; visual mesh filename=../meshes/head.stl scale=0.001 0.001 0.001
- added link left_elbow_link, mass 0.08453041843930957; collision mesh filename=../meshes/left_elbow.stl scale=0.001 0.001 0.001; visual mesh filename=../meshes/left_elbow.stl scale=0.001 0.001 0.001
- added link left_hand_link, mass 0.32306793312334026; collision mesh filename=../meshes/left_hand.stl scale=0.001 0.001 0.001; visual mesh filename=../meshes/left_hand.stl scale=0.001 0.001 0.001
- added link left_shoulder_pitch_link, mass 0.4197959811631081; collision mesh filename=../meshes/left_shoulder_pitch.stl scale=0.001 0.001 0.001; visual mesh filename=../meshes/left_shoulder_pitch.stl scale=0.001 0.001 0.001
- added link left_shoulder_roll_link, mass 0.4591563607035851; collision mesh filename=../meshes/left_shoulder_roll.stl scale=0.001 0.001 0.001; visual mesh filename=../meshes/left_shoulder_roll.stl scale=0.001 0.001 0.001
- added link left_shoulder_yaw_link, mass 0.4627321597109813; collision mesh filename=../meshes/left_shoulder_yaw.stl scale=0.001 0.001 0.001; visual mesh filename=../meshes/left_shoulder_yaw.stl scale=0.001 0.001 0.001
- added link neck_link, mass 0.39041587404351114; collision mesh filename=../meshes/neck.stl scale=0.001 0.001 0.001; visual mesh filename=../meshes/neck.stl scale=0.001 0.001 0.001
- added link right_elbow_link, mass 0.08452681925222644; collision mesh filename=../meshes/right_elbow.stl scale=0.001 0.001 0.001; visual mesh filename=../meshes/right_elbow.stl scale=0.001 0.001 0.001
- added link right_hand_link, mass 0.32306793312334026; collision mesh filename=../meshes/right_hand.stl scale=0.001 0.001 0.001; visual mesh filename=../meshes/right_hand.stl scale=0.001 0.001 0.001
- added link right_shoulder_pitch_link, mass 0.4285978598682473; collision mesh filename=../meshes/right_shoulder_pitch.stl scale=0.001 0.001 0.001; visual mesh filename=../meshes/right_shoulder_pitch.stl scale=0.001 0.001 0.001
- added link right_shoulder_roll_link, mass 0.45915238056305535; collision mesh filename=../meshes/right_shoulder_roll.stl scale=0.001 0.001 0.001; visual mesh filename=../meshes/right_shoulder_roll.stl scale=0.001 0.001 0.001
- added link right_shoulder_yaw_link, mass 0.4627321597115143; collision mesh filename=../meshes/right_shoulder_yaw.stl scale=0.001 0.001 0.001; visual mesh filename=../meshes/right_shoulder_yaw.stl scale=0.001 0.001 0.001
- added link torso_link, mass 3.2042605310287064; collision mesh filename=../meshes/torso.stl scale=0.001 0.001 0.001; visual mesh filename=../meshes/torso.stl scale=0.001 0.001 0.001
Joints:
- removed joint base_刚性-94
- removed joint base_旋转-91
- removed joint base_旋转-92
- removed joint base_旋转-93
- removed joint left_elbow_left-hand-joint
- removed joint left_shoulder_pitch_Left-Upper-Joint
- removed joint left_shoulder_roll_Left-Center-Joint
- removed joint left_shoulder_yaw_left-lower-joint
- removed joint neck_head-joint
- removed joint right_elbow_right-hand-joint
- removed joint right_shoulder_pitch_Right-Upper-Joint
- removed joint right_shoulder_roll_Right-Center-Joint
- removed joint right_shoulder_yaw_right-lower-joint
- removed joint torso_left-chest-joint
- removed joint torso_neck-joint
- removed joint torso_right-chest-joint
- added joint ball_x: type continuous, parent base_link, child ball_x_link, axis 1 0 0
- added joint ball_y: type continuous, parent ball_x_link, child ball_y_link, axis 0 1 0
- added joint ball_z: type continuous, parent ball_y_link, child ball_link, axis 0 0 1
- added joint base-91: type continuous, parent base_link, child omniwheel_base-v1_a, origin xyz=0.09652004 -1.5000000000000002e-07 0.13682553 rpy=3.141592653589793 0.7853981634093242 3.141592653589793, axis 1.1875833649810374e-11 0.0 1.0000003094489522
- added joint base-92: type continuous, parent base_link, child omniwheel_base-v1_b, origin xyz=-0.048260069999999995 0.08358868 0.13682553 rpy=2.394694060528722 -0.2705497629804707 -2.899028779496438, axis -3.230029243239674e-07 -4.7259469682092714e-07 0.999999749820805
- added joint base-93: type continuous, parent base_link, child omniwheel_base-v1_c, origin xyz=-0.048260069999999995 -0.08358898999999999 0.13682553 rpy=-2.394694060522079 -0.2705497629649148 2.8990287795064082, axis -3.229849821484443e-07 4.7260400443116524e-07 0.9999997498208049
- added joint head_joint: type continuous, parent neck_link, child head_link, origin xyz=0.0 -0.018 0.05200000000000003 rpy=3.141592653589793 -1.5707963267948966 0, axis -0.0 0.9999999999999999 4.652166535469666e-31
- added joint left_elbow_joint: type continuous, parent left_shoulder_yaw_link, child left_elbow_link, origin xyz=0.0 -0.125 0.01800000000000001 rpy=1.5707963267948966 -5.169878828456424e-26 1.5707963267948966, axis 5.169878828456423e-26 0.9999999999999999 9.386263146400684e-31
- added joint left_hand_joint: type fixed, parent left_elbow_link, child left_hand_link, origin xyz=-0.23800000000000004 -0.01800000000000001 0.0 rpy=-1.5707963267948966 -1.5707963267948966 0
- added joint left_shoulder_pitch_joint: type continuous, parent torso_link, child left_shoulder_pitch_link, origin xyz=0.009999999995371598 -0.10399999999958798 0.39000000000022866 rpy=-1.5707963267938403 1.186769372191522e-11 -3.141592653589793, axis 1.6816046190631742e-32 0.0 0.9999999999999999
- added joint left_shoulder_roll_joint: type revolute, parent left_shoulder_pitch_link, child left_shoulder_roll_link, origin xyz=0.018 0.0 0.05199999999999999 rpy=1.5707963267948966 -2.0194839173657902e-28 -1.5707963267948966, axis -3.323590376526234e-32 2.5849394142282115e-26 -1.0, limit lower=-0.174533 upper=2.356194 effort=1000000 velocity=1000000
- added joint left_shoulder_yaw_joint: type revolute, parent left_shoulder_roll_link, child left_shoulder_yaw_link, origin xyz=-0.13400000000000006 0.0 0.018 rpy=1.5707963267948966 1.5707963267948966 0, axis -1.2814691632297095e-31 -0.9999999999999999 2.5849394142282115e-26, limit lower=-1.570796 upper=1.570796 effort=1000000 velocity=1000000
- added joint neck_joint: type continuous, parent torso_link, child neck_link, origin xyz=0.009999999994374714 0.05500000000050074 0.4740000000000606 rpy=1.0564095652233624e-12 1.186769372191522e-11 -3.141592653589793, axis 0.0 0.0 1.0
- added joint right_elbow_joint: type continuous, parent right_shoulder_yaw_link, child right_elbow_link, origin xyz=0.0002528899999999999 -0.12499737000000004 -0.018016429999999986 rpy=1.5707963267948966 -2.584939414228211e-26 1.5707963267948966, axis 0.00014600000000000003 -0.999901 0.014049000000000002
- added joint right_hand_joint: type fixed, parent right_elbow_link, child right_hand_link, origin xyz=-0.2380026199999999 0.01796356000000003 -0.00025288999999999997 rpy=-1.5707963267948966 -1.5707963267948966 0
- added joint right_shoulder_pitch_joint: type continuous, parent torso_link, child right_shoulder_pitch_link, origin xyz=0.009999999995371598 0.214000000000412 0.3899999999998927 rpy=1.570796326795953 1.186769372191522e-11 -3.141592653589793, axis -1.6816046190631742e-32 0.0 0.9999999999999999
- added joint right_shoulder_roll_joint: type revolute, parent right_shoulder_pitch_link, child right_shoulder_roll_link, origin xyz=0.018 0.0 0.05199999999999998 rpy=-1.5707963267948966 -2.0194839173657907e-28 1.5707963267948966, axis -1.3173320852800765e-31 0.0 -0.9999999999999999, limit lower=-2.356194 upper=0.174533 effort=1000000 velocity=1000000
- added joint right_shoulder_yaw_joint: type revolute, parent right_shoulder_roll_link, child right_shoulder_yaw_link, origin xyz=-0.13400000000000006 1.9509999999982596e-05 0.018000000000000002 rpy=1.5707963267948966 1.5707963267948966 0, axis 0.0 -1.0 -0.00014600000000000003, limit lower=-1.570796 upper=1.570796 effort=1000000 velocity=1000000
- added joint torso_joint: type fixed, parent base_link, child torso_link, origin xyz=0.00999996 0.054999849999999996 0.44000037 rpy=1.0564095652233626e-12 1.186769372191522e-11 -3.141592653589793
