Commit message: modified:   LICENSE-CC-BY-NC-4.0.md 	modified:   README.md 	deleted:    ballbot_base_link.urdf 	deleted:    ballbot_floor.urdf 	modified:   hardware_code/damiao_mvp/SerialPort.h 	modified:   hardware_code/damiao_mvp/damiao.h 	modified:   hardware_code/damiao_mvp/test_damiao.cpp 	modified:   hardware_code/damiao_wrist.cpp 	modified:   hardware_code/inspire_hand.cpp 	modified:   hardware_code/zed_odometry.py 	modified:   images/H2O.gif 	modified:   images/H2O.webm 	modified:   images/OmniH2O.gif 	modified:   images/OmniH2O.webm 	modified:   images/hardware.png 	modified:   legged_gym/test.ipynb 	new file:   phc/phc/utils/motion_lib_ballbot.py 	modified:   phc/phc/utils/motion_lib_h1.py 	modified:   phc/phc/utils/torch_ballbot_batch.py 	modified:   phc/phc/utils/torch_h1_humanoid_batch.py 	modified:   resources/robots/ballbot/ballbot.xml 	deleted:    resources/robots/ballbot/meshes/FatRoller1_2.stl 	deleted:    resources/robots/ballbot/meshes/FatRoller1_3.stl 	deleted:    resources/robots/ballbot/meshes/FatRoller1_4.stl 	deleted:    resources/robots/ballbot/meshes/FatRoller1_5.stl 	deleted:    resources/robots/ballbot/meshes/FatRoller1_6.stl 	deleted:    resources/robots/ballbot/meshes/FatRoller2_1.stl 	deleted:    resources/robots/ballbot/meshes/FatRoller2_2.stl 	deleted:    resources/robots/ballbot/meshes/FatRoller2_3.stl 	deleted:    resources/robots/ballbot/meshes/FatRoller2_4.stl 	deleted:    resources/robots/ballbot/meshes/FatRoller2_5.stl 	deleted:    resources/robots/ballbot/meshes/FatRoller2_6.stl 	deleted:    resources/robots/ballbot/meshes/FatRoller3_1.stl 	deleted:    resources/robots/ballbot/meshes/FatRoller3_2.stl 	deleted:    resources/robots/ballbot/meshes/FatRoller3_3.stl 	deleted:    resources/robots/ballbot/meshes/FatRoller3_4.stl 	deleted:    resources/robots/ballbot/meshes/FatRoller3_5.stl 	deleted:    resources/robots/ballbot/meshes/FatRoller3_6.stl 	deleted:    resources/robots/ballbot/meshes/ThinRoller1_2.stl 	deleted:    resources/robots/ballbot/meshes/ThinRoller1_3.stl 	deleted:    resources/robots/ballbot/meshes/ThinRoller1_4.stl 	deleted:    resources/robots/ballbot/meshes/ThinRoller1_5.stl 	deleted:    resources/robots/ballbot/meshes/ThinRoller1_6.stl 	deleted:    resources/robots/ballbot/meshes/ThinRoller2_1.stl 	deleted:    resources/robots/ballbot/meshes/ThinRoller2_2.stl 	deleted:    resources/robots/ballbot/meshes/ThinRoller2_3.stl 	deleted:    resources/robots/ballbot/meshes/ThinRoller2_4.stl 	deleted:    resources/robots/ballbot/meshes/ThinRoller2_5.stl 	deleted:    resources/robots/ballbot/meshes/ThinRoller3_5.stl 	deleted:    resources/robots/ballbot/meshes/axle.stl 	renamed:    resources/robots/ballbot/meshes/ball.stl -> resources/robots/ballbot/meshes/ball_link.stl 	deleted:    resources/robots/ballbot/meshes/base.stl 	new file:   resources/robots/ballbot/meshes/base_link.stl 	deleted:    resources/robots/ballbot/meshes/fat_roller.stl 	deleted:    resources/robots/ballbot/meshes/fra2.stl 	deleted:    resources/robots/ballbot/meshes/fra3.stl 	deleted:    resources/robots/ballbot/meshes/fra4.stl 	deleted:    resources/robots/ballbot/meshes/fra5.stl 	deleted:    resources/robots/ballbot/meshes/frb1.stl 	deleted:    resources/robots/ballbot/meshes/frb2.stl 	deleted:    resources/robots/ballbot/meshes/frb3.stl 	deleted:    resources/robots/ballbot/meshes/frb4.stl 	deleted:    resources/robots/ballbot/meshes/frb5.stl 	deleted:    resources/robots/ballbot/meshes/frc1.stl 	deleted:    resources/robots/ballbot/meshes/frc2.stl 	deleted:    resources/robots/ballbot/meshes/frc3.stl 	deleted:    resources/robots/ballbot/meshes/frc4.stl 	deleted:    resources/robots/ballbot/meshes/frc5.stl 	deleted:    resources/robots/ballbot/meshes/head.stl 	new file:   resources/robots/ballbot/meshes/head_link.stl 	renamed:    resources/robots/ballbot/meshes/fra1.stl -> resources/robots/ballbot/meshes/large_roller_link.stl 	deleted:    resources/robots/ballbot/meshes/left_elbow.stl 	new file:   resources/robots/ballbot/meshes/left_elbow_link.stl 	deleted:    resources/robots/ballbot/meshes/left_hand.stl 	deleted:    resources/robots/ballbot/meshes/left_shoulder_pitch.stl 	new file:   resources/robots/ballbot/meshes/left_shoulder_pitch_link.stl 	deleted:    resources/robots/ballbot/meshes/left_shoulder_roll.stl 	new file:   resources/robots/ballbot/meshes/left_shoulder_roll_link.stl 	deleted:    resources/robots/ballbot/meshes/left_shoulder_yaw.stl 	new file:   resources/robots/ballbot/meshes/left_shoulder_yaw_link.stl 	deleted:    resources/robots/ballbot/meshes/neck.stl 	new file:   resources/robots/ballbot/meshes/neck_link.stl 	deleted:    resources/robots/ballbot/meshes/omniwheel_base-v1_b.stl 	deleted:    resources/robots/ballbot/meshes/omniwheel_base-v1_c.stl 	deleted:    resources/robots/ballbot/meshes/right_elbow.stl 	new file:   resources/robots/ballbot/meshes/right_elbow_link.stl 	deleted:    resources/robots/ballbot/meshes/right_hand.stl 	deleted:    resources/robots/ballbot/meshes/right_shoulder_pitch.stl 	new file:   resources/robots/ballbot/meshes/right_shoulder_pitch_link.stl 	deleted:    resources/robots/ballbot/meshes/right_shoulder_roll.stl 	new file:   resources/robots/ballbot/meshes/right_shoulder_roll_link.stl 	deleted:    resources/robots/ballbot/meshes/right_shoulder_yaw.stl 	new file:   resources/robots/ballbot/meshes/right_shoulder_yaw_link.stl 	renamed:    resources/robots/ballbot/meshes/tra1.stl -> resources/robots/ballbot/meshes/small_roller_link.stl 	deleted:    resources/robots/ballbot/meshes/thin_roller.stl 	deleted:    resources/robots/ballbot/meshes/thin_roller_2_6.stl 	deleted:    resources/robots/ballbot/meshes/thin_roller_3_1.stl 	deleted:    resources/robots/ballbot/meshes/thin_roller_3_2.stl 	deleted:    resources/robots/ballbot/meshes/thin_roller_3_3.stl 	deleted:    resources/robots/ballbot/meshes/thin_roller_3_4.stl 	deleted:    resources/robots/ballbot/meshes/thin_roller_3_6.stl 	deleted:    resources/robots/ballbot/meshes/torso.stl 	new file:   resources/robots/ballbot/meshes/torso_link.stl 	deleted:    resources/robots/ballbot/meshes/tra2.stl 	deleted:    resources/robots/ballbot/meshes/tra3.stl 	deleted:    resources/robots/ballbot/meshes/tra4.stl 	deleted:    resources/robots/ballbot/meshes/tra5.stl 	deleted:    resources/robots/ballbot/meshes/trb1.stl 	deleted:    resources/robots/ballbot/meshes/trb2.stl 	deleted:    resources/robots/ballbot/meshes/trb3.stl 	deleted:    resources/robots/ballbot/meshes/trb4.stl 	deleted:    resources/robots/ballbot/meshes/trb5.stl 	deleted:    resources/robots/ballbot/meshes/trc1.stl 	deleted:    resources/robots/ballbot/meshes/trc2.stl 	deleted:    resources/robots/ballbot/meshes/trc3.stl 	deleted:    resources/robots/ballbot/meshes/trc4.stl 	deleted:    resources/robots/ballbot/meshes/trc5.stl 	renamed:    resources/robots/ballbot/meshes/omniwheel_base-v1_a.stl -> resources/robots/ballbot/meshes/wheel_base_link.stl 	modified:   resources/robots/ballbot/urdf/ballbot.urdf 	modified:   resources/robots/pybullet_test.py 	modified:   scripts/data_process/grad_fit_ballbot.py 	modified:   scripts/data_process/grad_fit_ballbot_shape.py 	modified:   scripts/data_process/grad_fit_h1.py 	modified:   scripts/data_process/grad_fit_h1_shape.py 	modified:   scripts/joint_mokey_ballbot.py 	modified:   scripts/vis/vis_motion.py 	modified:   test.ipynb

File: resources/robots/ballbot/urdf/ballbot.urdf (robot description, URDF)
Before this commit: robot ballbot, 50 links, 49 joints
Links:
- removed link ball_link
- removed link ball_x_link
- removed link ball_y_link
- removed link fra1
- removed link fra2
- removed link fra3
- removed link fra4
- removed link fra5
- removed link frb1
- removed link frb2
- removed link frb3
- removed link frb4
- removed link frb5
- removed link frc1
- removed link frc2
- removed link frc3
- removed link frc4
- removed link frc5
- removed link left_hand_link
- removed link omniwheel_base-v1_a
- removed link omniwheel_base-v1_b
- removed link omniwheel_base-v1_c
- removed link right_hand_link
- removed link tra1
- removed link tra2
- removed link tra3
- removed link tra4
- removed link tra5
- removed link trb1
- removed link trb2
- removed link trb3
- removed link trb4
- removed link trb5
- removed link trc1
- removed link trc2
- removed link trc3
- removed link trc4
- removed link trc5
- added link large_roller_1_1_link, mass 0.026209434773783076; collision mesh filename=../meshes/large_roller_link.stl scale=0.001 0.001 0.001; visual mesh filename=../meshes/large_roller_link.stl scale=0.001 0.001 0.001
- added link large_roller_1_2_link, mass 0.026209434773783076; collision mesh filename=../meshes/large_roller_link.stl scale=0.001 0.001 0.001; visual mesh filename=../meshes/large_roller_link.stl scale=0.001 0.001 0.001
- added link large_roller_1_3_link, mass 0.026209434773783076; collision mesh filename=../meshes/large_roller_link.stl scale=0.001 0.001 0.001; visual mesh filename=../meshes/large_roller_link.stl scale=0.001 0.001 0.001
- added link large_roller_1_4_link, mass 0.026209434773783076; collision mesh filename=../meshes/large_roller_link.stl scale=0.001 0.001 0.001; visual mesh filename=../meshes/large_roller_link.stl scale=0.001 0.001 0.001
- added link large_roller_1_5_link, mass 0.026209434773783076; collision mesh filename=../meshes/large_roller_link.stl scale=0.001 0.001 0.001; visual mesh filename=../meshes/large_roller_link.stl scale=0.001 0.001 0.001
- added link large_roller_2_1_link, mass 0.026209434773783076; collision mesh filename=../meshes/large_roller_link.stl scale=0.001 0.001 0.001; visual mesh filename=../meshes/large_roller_link.stl scale=0.001 0.001 0.001
- added link large_roller_2_2_link, mass 0.026209434773783076; collision mesh filename=../meshes/large_roller_link.stl scale=0.001 0.001 0.001; visual mesh filename=../meshes/large_roller_link.stl scale=0.001 0.001 0.001
- added link large_roller_2_3_link, mass 0.026209434773783076; collision mesh filename=../meshes/large_roller_link.stl scale=0.001 0.001 0.001; visual mesh filename=../meshes/large_roller_link.stl scale=0.001 0.001 0.001
- added link large_roller_2_4_link, mass 0.026209434773783076; collision mesh filename=../meshes/large_roller_link.stl scale=0.001 0.001 0.001; visual mesh filename=../meshes/large_roller_link.stl scale=0.001 0.001 0.001
- added link large_roller_2_5_link, mass 0.026209434773783076; collision mesh filename=../meshes/large_roller_link.stl scale=0.001 0.001 0.001; visual mesh filename=../meshes/large_roller_link.stl scale=0.001 0.001 0.001
- added link large_roller_3_1_link, mass 0.026209434773783076; collision mesh filename=../meshes/large_roller_link.stl scale=0.001 0.001 0.001; visual mesh filename=../meshes/large_roller_link.stl scale=0.001 0.001 0.001
- added link large_roller_3_2_link, mass 0.026209434773783076; collision mesh filename=../meshes/large_roller_link.stl scale=0.001 0.001 0.001; visual mesh filename=../meshes/large_roller_link.stl scale=0.001 0.001 0.001
- added link large_roller_3_3_link, mass 0.026209434773783076; collision mesh filename=../meshes/large_roller_link.stl scale=0.001 0.001 0.001; visual mesh filename=../meshes/large_roller_link.stl scale=0.001 0.001 0.001
- added link large_roller_3_4_link, mass 0.026209434773783076; collision mesh filename=../meshes/large_roller_link.stl scale=0.001 0.001 0.001; visual mesh filename=../meshes/large_roller_link.stl scale=0.001 0.001 0.001
- added link large_roller_3_5_link, mass 0.026209434773783076; collision mesh filename=../meshes/large_roller_link.stl scale=0.001 0.001 0.001; visual mesh filename=../meshes/large_roller_link.stl scale=0.001 0.001 0.001
- added link small_roller_1_1_link, mass 0.014279541547129664; collision mesh filename=../meshes/small_roller_link.stl scale=0.001 0.001 0.001; visual mesh filename=../meshes/small_roller_link.stl scale=0.001 0.001 0.001
- added link small_roller_1_2_link, mass 0.014279541547129664; collision mesh filename=../meshes/small_roller_link.stl scale=0.001 0.001 0.001; visual mesh filename=../meshes/small_roller_link.stl scale=0.001 0.001 0.001
- added link small_roller_1_3_link, mass 0.014279541547129664; collision mesh filename=../meshes/small_roller_link.stl scale=0.001 0.001 0.001; visual mesh filename=../meshes/small_roller_link.stl scale=0.001 0.001 0.001
- added link small_roller_1_4_link, mass 0.014279541547129664; collision mesh filename=../meshes/small_roller_link.stl scale=0.001 0.001 0.001; visual mesh filename=../meshes/small_roller_link.stl scale=0.001 0.001 0.001
- added link small_roller_1_5_link, mass 0.014279541547129664; collision mesh filename=../meshes/small_roller_link.stl scale=0.001 0.001 0.001; visual mesh filename=../meshes/small_roller_link.stl scale=0.001 0.001 0.001
- added link small_roller_2_1_link, mass 0.014279541547129664; collision mesh filename=../meshes/small_roller_link.stl scale=0.001 0.001 0.001; visual mesh filename=../meshes/small_roller_link.stl scale=0.001 0.001 0.001
- added link small_roller_2_2_link, mass 0.014279541547129664; collision mesh filename=../meshes/small_roller_link.stl scale=0.001 0.001 0.001; visual mesh filename=../meshes/small_roller_link.stl scale=0.001 0.001 0.001
- added link small_roller_2_3_link, mass 0.014279541547129664; collision mesh filename=../meshes/small_roller_link.stl scale=0.001 0.001 0.001; visual mesh filename=../meshes/small_roller_link.stl scale=0.001 0.001 0.001
- added link small_roller_2_4_link, mass 0.014279541547129664; collision mesh filename=../meshes/small_roller_link.stl scale=0.001 0.001 0.001; visual mesh filename=../meshes/small_roller_link.stl scale=0.001 0.001 0.001
- added link small_roller_2_5_link, mass 0.014279541547129664; collision mesh filename=../meshes/small_roller_link.stl scale=0.001 0.001 0.001; visual mesh filename=../meshes/small_roller_link.stl scale=0.001 0.001 0.001
- added link small_roller_3_1_link, mass 0.014279541547129664; collision mesh filename=../meshes/small_roller_link.stl scale=0.001 0.001 0.001; visual mesh filename=../meshes/small_roller_link.stl scale=0.001 0.001 0.001
- added link small_roller_3_2_link, mass 0.014279541547129664; collision mesh filename=../meshes/small_roller_link.stl scale=0.001 0.001 0.001; visual mesh filename=../meshes/small_roller_link.stl scale=0.001 0.001 0.001
- added link small_roller_3_3_link, mass 0.014279541547129664; collision mesh filename=../meshes/small_roller_link.stl scale=0.001 0.001 0.001; visual mesh filename=../meshes/small_roller_link.stl scale=0.001 0.001 0.001
- added link small_roller_3_4_link, mass 0.014279541547129664; collision mesh filename=../meshes/small_roller_link.stl scale=0.001 0.001 0.001; visual mesh filename=../meshes/small_roller_link.stl scale=0.001 0.001 0.001
- added link small_roller_3_5_link, mass 0.014279541547129664; collision mesh filename=../meshes/small_roller_link.stl scale=0.001 0.001 0.001; visual mesh filename=../meshes/small_roller_link.stl scale=0.001 0.001 0.001
- added link wheel_base_1_link, mass 0.17443341496039455; collision mesh filename=../meshes/wheel_base_link.stl scale=0.001 0.001 0.001; visual mesh filename=../meshes/wheel_base_link.stl scale=0.001 0.001 0.001
- added link wheel_base_2_link, mass 0.17443341496039455; collision mesh filename=../meshes/wheel_base_link.stl scale=0.001 0.001 0.001; visual mesh filename=../meshes/wheel_base_link.stl scale=0.001 0.001 0.001
- added link wheel_base_3_link, mass 0.17443341496039455; collision mesh filename=../meshes/wheel_base_link.stl scale=0.001 0.001 0.001; visual mesh filename=../meshes/wheel_base_link.stl scale=0.001 0.001 0.001
- link base_link: geometry collision mesh filename=../meshes/base_link.stl scale=0.001 0.001 0.001; visual mesh filename=../meshes/base_link.stl scale=0.001 0.001 0.001
- link head_link: mass 1.0299685988699756 -> 0.41566857186457795; geometry collision mesh filename=../meshes/head_link.stl scale=0.001 0.001 0.001; visual mesh filename=../meshes/head_link.stl scale=0.001 0.001 0.001
- link left_elbow_link: mass 0.08453041843930957 -> 0.1558676529430366; geometry collision mesh filename=../meshes/left_elbow_link.stl scale=0.001 0.001 0.001; visual mesh filename=../meshes/left_elbow_link.stl scale=0.001 0.001 0.001
- link left_shoulder_pitch_link: mass 0.4197959811631081 -> 0.5647196059165264; geometry collision mesh filename=../meshes/left_shoulder_pitch_link.stl scale=0.001 0.001 0.001; visual mesh filename=../meshes/left_shoulder_pitch_link.stl scale=0.001 0.001 0.001
- link left_shoulder_roll_link: mass 0.4591563607035851 -> 0.41969396888718885; geometry collision mesh filename=../meshes/left_shoulder_roll_link.stl scale=0.001 0.001 0.001; visual mesh filename=../meshes/left_shoulder_roll_link.stl scale=0.001 0.001 0.001
- link left_shoulder_yaw_link: mass 0.4627321597109813 -> 0.42120157414587867; geometry collision mesh filename=../meshes/left_shoulder_yaw_link.stl scale=0.001 0.001 0.001; visual mesh filename=../meshes/left_shoulder_yaw_link.stl scale=0.001 0.001 0.001
- link neck_link: mass 0.39041587404351114 -> 0.6024876453871971; geometry collision mesh filename=../meshes/neck_link.stl scale=0.001 0.001 0.001; visual mesh filename=../meshes/neck_link.stl scale=0.001 0.001 0.001
- link right_elbow_link: mass 0.08452681925222644 -> 0.15586791529929014; geometry collision mesh filename=../meshes/right_elbow_link.stl scale=0.001 0.001 0.001; visual mesh filename=../meshes/right_elbow_link.stl scale=0.001 0.001 0.001
- link right_shoulder_pitch_link: mass 0.4285978598682473 -> 0.5647195174488359; geometry collision mesh filename=../meshes/right_shoulder_pitch_link.stl scale=0.001 0.001 0.001; visual mesh filename=../meshes/right_shoulder_pitch_link.stl scale=0.001 0.001 0.001
- link right_shoulder_roll_link: mass 0.45915238056305535 -> 0.41969396888718835; geometry collision mesh filename=../meshes/right_shoulder_roll_link.stl scale=0.001 0.001 0.001; visual mesh filename=../meshes/right_shoulder_roll_link.stl scale=0.001 0.001 0.001
- link right_shoulder_yaw_link: mass 0.4627321597115143 -> 0.31888998976294225; geometry collision mesh filename=../meshes/right_shoulder_yaw_link.stl scale=0.001 0.001 0.001; visual mesh filename=../meshes/right_shoulder_yaw_link.stl scale=0.001 0.001 0.001
- link torso_link: geometry collision mesh filename=../meshes/torso_link.stl scale=0.001 0.001 0.001; visual mesh filename=../meshes/torso_link.stl scale=0.001 0.001 0.001
Joints:
- removed joint ball_x
- removed joint ball_y
- removed joint ball_z
- removed joint base-91
- removed joint base-92
- removed joint base-93
- removed joint left_hand_joint
- removed joint omniwheel_base-v1_a_fraj1
- removed joint omniwheel_base-v1_a_fraj2
- removed joint omniwheel_base-v1_a_fraj3
- removed joint omniwheel_base-v1_a_fraj4
- removed joint omniwheel_base-v1_a_fraj5
- removed joint omniwheel_base-v1_a_traj1
- removed joint omniwheel_base-v1_a_traj2
- removed joint omniwheel_base-v1_a_traj3
- removed joint omniwheel_base-v1_a_traj4
- removed joint omniwheel_base-v1_a_traj5
- removed joint omniwheel_base-v1_b_frbj1
- removed joint omniwheel_base-v1_b_frbj2
- removed joint omniwheel_base-v1_b_frbj3
- removed joint omniwheel_base-v1_b_frbj4
- removed joint omniwheel_base-v1_b_frbj5
- removed joint omniwheel_base-v1_b_trbj1
- removed joint omniwheel_base-v1_b_trbj2
- removed joint omniwheel_base-v1_b_trbj3
- removed joint omniwheel_base-v1_b_trbj4
- removed joint omniwheel_base-v1_b_trbj5
- removed joint omniwheel_base-v1_c_frcj1
- removed joint omniwheel_base-v1_c_frcj2
- removed joint omniwheel_base-v1_c_frcj3
- removed joint omniwheel_base-v1_c_frcj4
- removed joint omniwheel_base-v1_c_frcj5
- removed joint omniwheel_base-v1_c_trcj1
- removed joint omniwheel_base-v1_c_trcj2
- removed joint omniwheel_base-v1_c_trcj3
- removed joint omniwheel_base-v1_c_trcj4
- removed joint omniwheel_base-v1_c_trcj5
- removed joint right_hand_joint
- added joint large_roller_1_1_joint: type continuous, parent wheel_base_1_link, child large_roller_1_1_link, origin xyz=-0.024816852937422418 -0.027089400000000003 0.028500002455628823 rpy=-2.251011303687431 0.4286319892053053 -1.0962147441310643, axis -0.8988079227928 0.4156269999999999 0.13927895513282618, limit effort=1000 velocity=1000
- added joint large_roller_1_2_joint: type continuous, parent wheel_base_1_link, child large_roller_1_2_link, origin xyz=-0.03343237630968773 0.01523114 0.02849999538466332 rpy=2.251011303687432 0.42863198920530315 1.0962147441310672, axis 0.8988079227928003 0.4156269999999999 -0.13927895513282312, limit effort=1000 velocity=1000
- added joint large_roller_1_3_joint: type continuous, parent wheel_base_1_link, child large_roller_1_3_link, origin xyz=0.004154506898250645 0.03650276 0.028499995384216957 rpy=1.2710877270196506 0.7375795500064168 -0.43073080773682754, axis 0.7350760607027366 0.6724989999999998 0.08607901179583019, limit effort=1000 velocity=1000
- added joint large_roller_1_4_joint: type continuous, parent wheel_base_1_link, child large_roller_1_4_link, origin xyz=0.03599999416993798 0.0073288 0.02849999538383877 rpy=-9.103828801926282e-15 0.7853981633855724 3.141592653589793, axis -0.0 0.9999999999999998 9.10382880192628e-15, limit effort=1000 velocity=1000
- added joint large_roller_1_5_joint: type continuous, parent wheel_base_1_link, child large_roller_1_5_link, origin xyz=0.018094706967410338 -0.031973310000000005 0.02849999538405141 rpy=-1.2710877270196352 0.7375795500064116 0.43073080773685035, axis -0.735076060702738 0.6724989999999998 -0.08607901179581726, limit effort=1000 velocity=1000
- added joint large_roller_2_1_joint: type continuous, parent wheel_base_2_link, child large_roller_2_1_link, origin xyz=0.004154508416893679 0.036502762357123186 0.028500004501358474 rpy=2.345148039247225 -0.14755057546463826 -0.23841317140416993, axis 0.9862981194264782 -0.05188099999999996 0.15660385794670795, limit effort=1000 velocity=1000
- added joint large_roller_2_2_joint: type continuous, parent wheel_base_2_link, child large_roller_2_2_link, origin xyz=0.03600000147244053 0.007328805131328302 0.02850000144188761 rpy=-2.0943951023971557 0.7853981634042961 1.1831996401341272, axis -0.654654 0.755929 6.902829446930878e-15, limit effort=1000 velocity=1000
- added joint large_roller_2_3_joint: type continuous, parent wheel_base_2_link, child large_roller_2_3_link, origin xyz=0.018094715702264175 -0.03197330200954152 0.028500004810741393 rpy=-0.981089858144548 -0.5532824127559389 0.2781297332436009, axis -0.8502521515849303 -0.45647999999999994 0.26210257757831523, limit effort=1000 velocity=1000
- added joint large_roller_2_4_joint: type continuous, parent wheel_base_2_link, child large_roller_2_4_link, origin xyz=-0.02481684456202 -0.027089383607755906 0.028500002294045236 rpy=-0.8305477513526444 0.291726533746681 -0.692597592885106, axis -0.928003000850887 0.372534 -0.00538495735809937, limit effort=1000 velocity=1000
- added joint large_roller_2_5_joint: type continuous, parent wheel_base_2_link, child large_roller_2_5_link, origin xyz=-0.03343237205306998 0.015231149913756249 0.028499996692232986 rpy=1.6749465668843488 -0.7799349548695472 1.0356401919704166, axis 0.7078767578344132 -0.686718 0.16531603443961382, limit effort=1000 velocity=1000
- added joint large_roller_3_1_joint: type continuous, parent wheel_base_3_link, child large_roller_3_1_link, origin xyz=0.018094718392606443 -0.03197330995039234 0.02849999769379311 rpy=-2.345148039252087 -0.14755057544499312 0.23841317140137927, axis -0.9862981194264809 -0.051881 -0.15660385794669068, limit effort=1000 velocity=1000
- added joint large_roller_3_2_joint: type continuous, parent wheel_base_3_link, child large_roller_3_2_link, origin xyz=-0.024816844262084317 -0.027089399688969173 0.02850000150228821 rpy=-1.674946566912737 -0.7799349548684031 -1.0356401919539688, axis -0.7078767578344138 -0.6867180000000002 -0.1653160344396113, limit effort=1000 velocity=1000
- added joint large_roller_3_3_joint: type continuous, parent wheel_base_3_link, child large_roller_3_3_link, origin xyz=-0.03343237131459437 0.01523114254782195 0.028499994740362952 rpy=0.8305477513571284 0.29172653376643465 0.69259759288288, axis 0.9280030008508872 0.37253400000000003 0.005384957358102466, limit effort=1000 velocity=1000
- added joint large_roller_3_4_joint: type continuous, parent wheel_base_3_link, child large_roller_3_4_link, origin xyz=0.004154512505998164 0.036502753201079444 0.02849999368388332 rpy=0.9810898581282296 -0.5532824127412317 -0.2781297332385313, axis 0.850252151584935 -0.4564800000000001 -0.2621025775783002, limit effort=1000 velocity=1000
- added joint large_roller_3_5_joint: type continuous, parent wheel_base_3_link, child large_roller_3_5_link, origin xyz=0.03600000327340246 0.0073287982382078815 0.02849999667769728 rpy=2.0943951023686704 0.7853981634024605 -1.183199640157774, axis 0.6546540000000001 0.7559290000000002 6.923810691450427e-15, limit effort=1000 velocity=1000
- added joint small_roller_1_1_joint: type continuous, parent wheel_base_1_link, child small_roller_1_1_link, origin xyz=0.0001695642064670011 -0.043165049999999996 0.02849999538426426 rpy=1.2710877270196437 0.7375795500064146 -0.4307308077368376, axis 0.7350760607027372 0.6724989999999998 0.0860790117958245, limit effort=1000 velocity=1000
- added joint small_roller_1_2_joint: type continuous, parent wheel_base_1_link, child small_roller_1_2_link, origin xyz=-0.04100000278757364 -0.013499999999999998 0.028499995384753184 rpy=-1.1538402495141857e-15 0.7853981633855724 3.141592653589793, axis -0.0 0.9999999999999998 1.1538402495141855e-15, limit effort=1000 velocity=1000
- added joint small_roller_1_3_joint: type continuous, parent wheel_base_1_link, child small_roller_1_3_link, origin xyz=-0.025508961983779985 0.03482159 0.028499995384569227 rpy=-1.2710877270196292 0.7375795500064096 0.43073080773685857, axis -0.7350760607027388 0.6724989999999997 -0.08607901179581272, limit effort=1000 velocity=1000
- added joint small_roller_1_4_joint: type continuous, parent wheel_base_1_link, child small_roller_1_4_link, origin xyz=0.025234590411220878 0.03502092 0.028499995383966616 rpy=-2.251011303687428 0.4286319892053099 -1.096214744131059, axis -0.8988079227927989 0.4156270000000004 0.139278955132832, limit effort=1000 velocity=1000
- added joint small_roller_1_5_joint: type continuous, parent wheel_base_1_link, child small_roller_1_5_link, origin xyz=0.0411047960132224 -0.01317747 0.028499995383778124 rpy=2.251011303687434 0.4286319892052995 1.0962147441310732, axis 0.8988079227928011 0.4156270000000004 -0.13927895513281718, limit effort=1000 velocity=1000
- added joint small_roller_2_1_joint: type continuous, parent wheel_base_2_link, child small_roller_2_1_link, origin xyz=-0.025508955582839672 0.034821589203660644 0.02850000392994919 rpy=-0.9810898581445507 -0.5532824127559426 0.2781297332436071, axis -0.8502521515849286 -0.45647999999999994 0.2621025775783209, limit effort=1000 velocity=1000
- added joint small_roller_2_2_joint: type continuous, parent wheel_base_2_link, child small_roller_2_2_link, origin xyz=0.025234600672920333 0.03502093596364762 0.028500002448176104 rpy=-0.8305477513526424 0.29172653374667695 -0.6925975928851004, axis -0.9280030008508868 0.3725340000000005 -0.00538495735809335, limit effort=1000 velocity=1000
- added joint small_roller_2_3_joint: type continuous, parent wheel_base_2_link, child small_roller_2_3_link, origin xyz=0.041104797366851076 -0.013177461501547754 0.028500003374909228 rpy=1.6749465668843422 -0.7799349548695474 1.035640191970426, axis 0.7078767578344124 -0.6867179999999997 0.16531603443961818, limit effort=1000 velocity=1000
- added joint small_roller_2_4_joint: type continuous, parent wheel_base_2_link, child small_roller_2_4_link, origin xyz=0.00016956977258599792 -0.043165045410434325 0.028500001046657317 rpy=2.3451480392472255 -0.147550575464633 -0.23841317140417564, axis 0.9862981194264795 -0.05188100000000013 0.15660385794670031, limit effort=1000 velocity=1000
- added joint small_roller_2_5_joint: type continuous, parent wheel_base_2_link, child small_roller_2_5_link, origin xyz=-0.04099999158431564 -0.013499994029705356 0.02849999635238339 rpy=-2.094395102397147 0.7853981634042961 1.1831996401341272, axis -0.654654 0.755929 1.1304771800368233e-15, limit effort=1000 velocity=1000
- added joint small_roller_3_1_joint: type continuous, parent wheel_base_3_link, child small_roller_3_1_link, origin xyz=0.04110480062647349 -0.013177470584983126 0.02849999475137443 rpy=0.8305477513571293 0.2917265337664395 0.6925975928828846, axis 0.9280030008508868 0.37253400000000053 0.005384957358108599, limit effort=1000 velocity=1000
- added joint small_roller_3_2_joint: type continuous, parent wheel_base_3_link, child small_roller_3_2_link, origin xyz=0.00016957096083211276 -0.043165055510583306 0.0284999979042035 rpy=0.981089858128233 -0.553282412741236 -0.27812973323853873, axis 0.850252151584933 -0.4564800000000001 -0.26210257757830696, limit effort=1000 velocity=1000
- added joint small_roller_3_3_joint: type continuous, parent wheel_base_3_link, child small_roller_3_3_link, origin xyz=-0.040999993661270814 -0.013499998840550198 0.028500001849578818 rpy=2.094395102368678 0.7853981634024605 -1.183199640157774, axis 0.6546540000000001 0.7559290000000002 6.769091654718352e-16, limit effort=1000 velocity=1000
- added joint small_roller_3_4_joint: type continuous, parent wheel_base_3_link, child small_roller_3_4_link, origin xyz=-0.025508955975381716 0.03482158427873564 0.028500004970328466 rpy=-2.3451480392520874 -0.1475505754449887 0.23841317140138402, axis -0.9862981194264822 -0.05188100000000017 -0.15660385794668433, limit effort=1000 velocity=1000
- added joint small_roller_3_5_joint: type continuous, parent wheel_base_3_link, child small_roller_3_5_link, origin xyz=0.025234601011656085 0.035020923992376 0.02850000155286571 rpy=-1.674946566912743 -0.7799349548684019 -1.0356401919539597, axis -0.7078767578344153 -0.6867179999999998 -0.16531603443960638, limit effort=1000 velocity=1000
- added joint wheel_base_1_joint: type continuous, parent base_link, child wheel_base_1_link, origin xyz=0.09652004 -1.5000000000000002e-07 0.13682553 rpy=3.141592653589793 0.7853981634093242 3.141592653589793, axis 1.1875833649810374e-11 0.0 1.0000003094489522, limit effort=1000 velocity=1000
- added joint wheel_base_2_joint: type continuous, parent base_link, child wheel_base_2_link, origin xyz=-0.048260069999999995 0.08358868 0.13682553 rpy=2.394694060528722 -0.2705497629804707 -2.899028779496438, axis -3.230029243239674e-07 -4.7259469682092714e-07 0.999999749820805, limit effort=1000 velocity=1000
- added joint wheel_base_3_joint: type continuous, parent base_link, child wheel_base_3_link, origin xyz=-0.048260069999999995 -0.08358898999999999 0.13682553 rpy=-2.394694060522079 -0.2705497629649148 2.8990287795064082, axis -3.229849821484443e-07 4.7260400443116524e-07 0.9999997498208049, limit effort=1000 velocity=1000
- joint head_joint: axis -0.0 0.9999999999999999 4.652166535469666e-31 -> 0.0 0.0 1.0; limit (none) -> lower=-3.141592653589793 upper=3.141592653589793 effort=1000 velocity=1000; origin xyz=0.0 -0.018 0.05200000000000003 rpy=3.141592653589793 -1.5707963267948966 0 -> xyz=0.0 -0.018 0.05200000000000003 rpy=1.5707963267948966 1.1750542820509288e-48 -1.6816046190631745e-32; type continuous -> revolute
- joint left_elbow_joint: axis 5.169878828456423e-26 0.9999999999999999 9.386263146400684e-31 -> 0.0 0.0 1.0; limit (none) -> lower=-3.141592653589793 upper=3.141592653589793 effort=1000 velocity=1000; origin xyz=0.0 -0.125 0.01800000000000001 rpy=1.5707963267948966 -5.169878828456424e-26 1.5707963267948966 -> xyz=0.0 -0.125 0.01800000000000001 rpy=1.2722748679404478e-26 1.3552292526152156e-58 -1.0616594778908991e-32; type continuous -> revolute
- joint left_shoulder_pitch_joint: axis 1.6816046190631742e-32 0.0 0.9999999999999999 -> 0.0 0.0 1.0; limit (none) -> lower=-3.141592653589793 upper=3.141592653589793 effort=1000 velocity=1000; type continuous -> revolute
- joint left_shoulder_roll_joint: axis -3.323590376526234e-32 2.5849394142282115e-26 -1.0 -> 0.0 0.0 1.0; limit lower=-0.174533 upper=2.356194 effort=1000000 velocity=1000000 -> lower=-3.141592653589793 upper=3.141592653589793 effort=1000 velocity=1000; origin xyz=0.018 0.0 0.05199999999999999 rpy=1.5707963267948966 -2.0194839173657902e-28 -1.5707963267948966 -> xyz=0.018 0.0 0.05199999999999999 rpy=1.5707963267948966 2.173422598490853e-58 -1.5707963267948966
- joint left_shoulder_yaw_joint: axis -1.2814691632297095e-31 -0.9999999999999999 2.5849394142282115e-26 -> 0.0 1.0 0.0; limit lower=-1.570796 upper=1.570796 effort=1000000 velocity=1000000 -> lower=-3.141592653589793 upper=3.141592653589793 effort=1000 velocity=1000
- joint neck_joint: limit (none) -> lower=-3.141592653589793 upper=3.141592653589793 effort=1000 velocity=1000; type continuous -> revolute
- joint right_elbow_joint: axis 0.00014600000000000003 -0.999901 0.014049000000000002 -> 0.0 0.0 1.0; limit (none) -> lower=-3.141592653589793 upper=3.141592653589793 effort=1000 velocity=1000; origin xyz=0.0002528899999999999 -0.12499737000000004 -0.018016429999999986 rpy=1.5707963267948966 -2.584939414228211e-26 1.5707963267948966 -> xyz=0.0 -0.125 -0.01800000000000001 rpy=-3.141592653589793 -5.191029131268521e-57 4.029163933488661e-31; type continuous -> revolute
- joint right_shoulder_pitch_joint: axis -1.6816046190631742e-32 0.0 0.9999999999999999 -> 0.0 0.0 1.0; limit (none) -> lower=-3.141592653589793 upper=3.141592653589793 effort=1000 velocity=1000; type continuous -> revolute
- joint right_shoulder_roll_joint: axis -1.3173320852800765e-31 0.0 -0.9999999999999999 -> 0.0 0.0 1.0; limit lower=-2.356194 upper=0.174533 effort=1000000 velocity=1000000 -> lower=-3.141592653589793 upper=3.141592653589793 effort=1000 velocity=1000; origin xyz=0.018 0.0 0.05199999999999998 rpy=-1.5707963267948966 -2.0194839173657907e-28 1.5707963267948966 -> xyz=0.018 0.0 0.05199999999999998 rpy=1.5707963267948966 2.0194839173657902e-28 1.5707963267948966
- joint right_shoulder_yaw_joint: axis 0.0 -1.0 -0.00014600000000000003 -> 0.0 1.0 0.0; limit lower=-1.570796 upper=1.570796 effort=1000000 velocity=1000000 -> lower=-3.141592653589793 upper=3.141592653589793 effort=1000 velocity=1000; origin xyz=-0.13400000000000006 1.9509999999982596e-05 0.018000000000000002 rpy=1.5707963267948966 1.5707963267948966 0 -> xyz=-0.13400000000000006 0.0 -0.018 rpy=-1.5707963267948966 -1.5707963267948966 0
